File: pcb/Bricoleur-pcb/Bricoleur-pcb.kicad_pcb (KiCad board)
At the start: 2 copper layers, 124.5 x 66 mm, 78 parts, among them J1 USB_B_Micro, J2 Conn_02x10_Odd_Even, J3 Conn_02x03_Odd_Even, J4 Conn_02x03_Odd_Even, SW2 SW_Push, SW3 SW_Push, SW4 SW_Push, SW5 SW_Push, U1 Ultrasonic-LV-EZ0, U11 SW_DP3T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

Commit message: Pcb finished???
Other:
- board text added: "BRICOLEUR"
- board text added: "Richard Bachmann Fritz-Olav Myrvang Valentin Plotkin Eirik Vale Aase Joakim Lier Marius Kohmann Ola Toft Eirik Smithsen Einar Hov Mathias Lundteigen Mohus"
Changed lines of the file:
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@@
   (general
     (thickness 1.6)
-    (drawings 131)
+    (drawings 133)
     (tracks 887)
     (zones 0)
@@
   (page A4)
   (layers
-    (0 F.Cu jumper hide)
-    (31 B.Cu signal hide)
+    (0 F.Cu jumper)
+    (31 B.Cu signal)
     (32 B.Adhes user)
     (33 F.Adhes user)
@@
       (net 24 "Net-(R13-Pad2)"))
   )
+  (gr_text "Richard Bachmann\nFritz-Olav Myrvang\nValentin Plotkin\nEirik Vale Aase\nJoakim Lier\nMarius Kohmann\nOla Toft\nEirik Smithsen\nEinar Hov\nMathias Lundteigen Mohus\n" (at 39.6937 150.4695 270) (layer F.SilkS)
+    (effects (font (size 1 1) (thickness 0.15)))
+  )
+  (gr_text BRICOLEUR (at 33.8517 122.1485 270) (layer F.SilkS)
+    (effects (font (size 2 2) (thickness 0.15)))
+  )
   (gr_line (start 33.3437 132.6895) (end 38.4237 137.7695) (layer F.SilkS) (width 0.15))
